Commit message: Added dynamics param in urdf

File: urdf/inc/ur_common.xacro (robot description, xacro)
@@ -20,4 +20,13 @@
     </inertial>
   </xacro:macro>
+  <!-- <xacro:macro name="cylinder_inertial" params="radius length mass *origin">
+    <inertial>
+      <mass value="2" />
+      <xacro:insert_block name="origin" />
+      <inertia ixx="0.01" ixy="0.0" ixz="0.0"
+        iyy="0.01" iyz="0.0"
+        izz="0.01" />
+    </inertial>
+  </xacro:macro> -->
   <xacro:macro name="get_visual_params" params="name:=^ type:=^" >
     <xacro:property name="visual_params" value="${sec_mesh_files[name][type]}" scope="parent"/>

File: urdf/ur_macro.xacro (robot description, xacro)
@@ -167,5 +167,6 @@
       </collision>
       <xacro:cylinder_inertial radius="${upperarm_inertia_radius}" length="${upperarm_inertia_length}" mass="${upper_arm_mass}">
-        <origin xyz="${-0.5 * upperarm_inertia_length} 0.0 ${upper_arm_inertia_offset}" rpy="0 ${pi/2} 0" />
+        <!-- <origin xyz="${-0.5 * upperarm_inertia_length} 0.0 ${upper_arm_inertia_offset}" rpy="0 ${pi/2} 0" /> -->
+        <origin xyz="0 0 0" rpy="0 0 0" />
       </xacro:cylinder_inertial>
     </link>
@@ -184,5 +185,6 @@
       </collision>
       <xacro:cylinder_inertial radius="${forearm_inertia_radius}" length="${forearm_inertia_length}"  mass="${forearm_mass}">
-        <origin xyz="${-0.5 * forearm_inertia_length} 0.0 ${elbow_offset}" rpy="0 ${pi/2} 0" />
+        <!-- <origin xyz="${-0.5 * forearm_inertia_length} 0.0 ${elbow_offset}" rpy="0 ${pi/2} 0" /> -->
+        <origin xyz="0 0 0" rpy="0 0 0" />
       </xacro:cylinder_inertial>
     </link>
@@ -238,5 +240,6 @@
       </collision>
       <xacro:cylinder_inertial radius="${wrist_3_inertia_radius}" length="${wrist_3_inertia_length}"  mass="${wrist_3_mass}">
-        <origin xyz="0.0 0.0 ${-0.5 * wrist_3_inertia_length}" rpy="0 0 0" />
+        <!-- <origin xyz="0.0 0.0 ${-0.5 * wrist_3_inertia_length}" rpy="0 0 0" /> -->
+        <origin xyz="0 0 0" rpy="0 0 0" />
       </xacro:cylinder_inertial>
     </link>
@@ -268,5 +271,6 @@
          <safety_controller soft_lower_limit="${shoulder_pan_lower_limit + safety_pos_margin}" soft_upper_limit="${shoulder_pan_upper_limit - safety_pos_margin}" k_position="${safety_k_position}" k_velocity="0.0"/>
       </xacro:if>
-      <dynamics damping="0" friction="0"/>
+      <dynamics damping="50" friction="5"/>
+      <!-- <dynamics damping="0" friction="0"/> -->
     </joint>
     <joint name="${prefix}shoulder_lift_joint" type="revolute">
@@ -280,5 +284,6 @@
          <safety_controller soft_lower_limit="${shoulder_lift_lower_limit + safety_pos_margin}" soft_upper_limit="${shoulder_lift_upper_limit - safety_pos_margin}" k_position="${safety_k_position}" k_velocity="0.0"/>
       </xacro:if>
-      <dynamics damping="0" friction="0"/>
+      <dynamics damping="50" friction="5"/>
+      <!-- <dynamics damping="0" friction="0"/> -->
     </joint>
     <joint name="${prefix}elbow_joint" type="revolute">
@@ -292,5 +297,6 @@
          <safety_controller soft_lower_limit="${elbow_joint_lower_limit + safety_pos_margin}" soft_upper_limit="${elbow_joint_upper_limit - safety_pos_margin}" k_position="${safety_k_position}" k_velocity="0.0"/>
       </xacro:if>
-      <dynamics damping="0" friction="0"/>
+      <dynamics damping="50" friction="5"/>
+      <!-- <dynamics damping="0" friction="0"/> -->
     </joint>
     <joint name="${prefix}wrist_1_joint" type="revolute">
@@ -304,5 +310,6 @@
          <safety_controller soft_lower_limit="${wrist_1_lower_limit + safety_pos_margin}" soft_upper_limit="${wrist_1_upper_limit - safety_pos_margin}" k_position="${safety_k_position}" k_velocity="0.0"/>
       </xacro:if>
-      <dynamics damping="0" friction="0"/>
+      <dynamics damping="10" friction="1"/>
+      <!-- <dynamics damping="0" friction="0"/> -->
     </joint>
     <joint name="${prefix}wrist_2_joint" type="revolute">
@@ -316,5 +323,6 @@
          <safety_controller soft_lower_limit="${wrist_2_lower_limit + safety_pos_margin}" soft_upper_limit="${wrist_2_upper_limit - safety_pos_margin}" k_position="${safety_k_position}" k_velocity="0.0"/>
       </xacro:if>
-      <dynamics damping="0" friction="0"/>
+      <dynamics damping="10" friction="1"/>
+      <!-- <dynamics damping="0" friction="0"/> -->
     </joint>
     <joint name="${prefix}wrist_3_joint" type="revolute">
@@ -328,5 +336,6 @@
          <safety_controller soft_lower_limit="${wrist_3_lower_limit + safety_pos_margin}" soft_upper_limit="${wrist_3_upper_limit - safety_pos_margin}" k_position="${safety_k_position}" k_velocity="0.0"/>
       </xacro:if>
-      <dynamics damping="0" friction="0"/>
+      <dynamics damping="10" friction="1"/>
+      <!-- <dynamics damping="0" friction="0"/> -->
     </joint>
     <link name="${prefix}ft_frame"/>
